Commit message: feat: add SLAM and RViz launch files, standardize base_footprint frame, and update hardware controller configurations.

File: ros2/src/uet_amr_description/urdf/materials.xacro (robot description, xacro)
@@ -2,5 +2,5 @@
 <robot name="uet_amr" xmlns:xacro="http://www.ros.org/wiki/xacro" >
 <material name="silver">
-  <color rgba="0.700 0.700 0.700 1.000"/>
+  <color rgba="0.55 0.58 0.62 1.000"/>
 </material>
 </robot>

File: ros2/src/uet_amr_description/urdf/uet_amr.xacro (robot description, xacro)
@@ -10,4 +10,11 @@
 </xacro:unless>
 <xacro:include filename="$(find uet_amr_description)/urdf/uet_amr.gazebo" />
+<link name="base_footprint">
+</link>
+<joint name="base_footprint_joint" type="fixed">
+    <parent link="base_footprint"/>
+    <child link="base_link"/>
+    <origin xyz="0 0 0.163" rpy="0 0 0"/>
+</joint>
 <link name="base_link">
   <inertial>
@@ -19,5 +26,5 @@
     <origin xyz="0 0 0" rpy="0 0 0"/>
     <geometry>
-      <mesh filename="file://$(find uet_amr_description)/meshes/base_link.stl" scale="0.001 0.001 0.001"/>
+      <mesh filename="package://uet_amr_description/meshes/base_link.stl" scale="0.001 0.001 0.001"/>
     </geometry>
     <material name="silver"/>
@@ -26,14 +33,7 @@
     <origin xyz="0 0 0" rpy="0 0 0"/>
     <geometry>
-      <mesh filename="file://$(find uet_amr_description)/meshes/base_link.stl" scale="0.001 0.001 0.001"/>
-    </geometry>
-  </collision>
-</link>
-<joint name="base_footprint_joint" type="fixed">
-    <parent link="base_link"/>
-    <child link="base_footprint"/>
-    <origin xyz="0 0 0" rpy="0 0 0"/>
-</joint>
-<link name="base_footprint">
+      <mesh filename="package://uet_amr_description/meshes/base_link.stl" scale="0.001 0.001 0.001"/>
+    </geometry>
+  </collision>
 </link>
 <link name="left_wheel_1">
@@ -46,5 +46,5 @@
     <origin xyz="-0.001978 -0.151669 0.077157" rpy="0 0 0"/>
     <geometry>
-      <mesh filename="file://$(find uet_amr_description)/meshes/left_wheel_1.stl" scale="0.001 0.001 0.001"/>
+      <mesh filename="package://uet_amr_description/meshes/left_wheel_1.stl" scale="0.001 0.001 0.001"/>
     </geometry>
     <material name="silver"/>
@@ -53,5 +53,5 @@
     <origin xyz="-0.001978 -0.151669 0.077157" rpy="0 0 0"/>
     <geometry>
-      <mesh filename="file://$(find uet_amr_description)/meshes/left_wheel_1.stl" scale="0.001 0.001 0.001"/>
+      <mesh filename="package://uet_amr_description/meshes/left_wheel_1.stl" scale="0.001 0.001 0.001"/>
     </geometry>
   </collision>
@@ -66,5 +66,5 @@
     <origin xyz="-0.002833 0.152327 0.078549" rpy="0 0 0"/>
     <geometry>
-      <mesh filename="file://$(find uet_amr_description)/meshes/right_wheel_1.stl" scale="0.001 0.001 0.001"/>
+      <mesh filename="package://uet_amr_description/meshes/right_wheel_1.stl" scale="0.001 0.001 0.001"/>
     </geometry>
     <material name="silver"/>
@@ -73,5 +73,5 @@
     <origin xyz="-0.002833 0.152327 0.078549" rpy="0 0 0"/>
     <geometry>
-      <mesh filename="file://$(find uet_amr_description)/meshes/right_wheel_1.stl" scale="0.001 0.001 0.001"/>
+      <mesh filename="package://uet_amr_description/meshes/right_wheel_1.stl" scale="0.001 0.001 0.001"/>
     </geometry>
   </collision>
@@ -86,5 +86,5 @@
     <origin xyz="0.213493 -0.141254 0.064203" rpy="0 0 0"/>
     <geometry>
-      <mesh filename="file://$(find uet_amr_description)/meshes/bl_caster_1.stl" scale="0.001 0.001 0.001"/>
+      <mesh filename="package://uet_amr_description/meshes/bl_caster_1.stl" scale="0.001 0.001 0.001"/>
     </geometry>
     <material name="silver"/>
@@ -93,5 +93,5 @@
     <origin xyz="0.213493 -0.141254 0.064203" rpy="0 0 0"/>
     <geometry>
-      <mesh filename="file://$(find uet_amr_description)/meshes/bl_caster_1.stl" scale="0.001 0.001 0.001"/>
+      <mesh filename="package://uet_amr_description/meshes/bl_caster_1.stl" scale="0.001 0.001 0.001"/>
     </geometry>
   </collision>
@@ -106,5 +106,5 @@
     <origin xyz="0.212694 0.143242 0.065506" rpy="0 0 0"/>
     <geometry>
-      <mesh filename="file://$(find uet_amr_description)/meshes/br_caster_1.stl" scale="0.001 0.001 0.001"/>
+      <mesh filename="package://uet_amr_description/meshes/br_caster_1.stl" scale="0.001 0.001 0.001"/>
     </geometry>
     <material name="silver"/>
@@ -113,5 +113,5 @@
     <origin xyz="0.212694 0.143242 0.065506" rpy="0 0 0"/>
     <geometry>
-      <mesh filename="file://$(find uet_amr_description)/meshes/br_caster_1.stl" scale="0.001 0.001 0.001"/>
+      <mesh filename="package://uet_amr_description/meshes/br_caster_1.stl" scale="0.001 0.001 0.001"/>
     </geometry>
   </collision>
@@ -126,5 +126,5 @@
     <origin xyz="-0.217505 -0.142465 0.064201" rpy="0 0 0"/>
     <geometry>
-      <mesh filename="file://$(find uet_amr_description)/meshes/fl_caster_1.stl" scale="0.001 0.001 0.001"/>
+      <mesh filename="package://uet_amr_description/meshes/fl_caster_1.stl" scale="0.001 0.001 0.001"/>
     </geometry>
     <material name="silver"/>
@@ -133,5 +133,5 @@
     <origin xyz="-0.217505 -0.142465 0.064201" rpy="0 0 0"/>
     <geometry>
-      <mesh filename="file://$(find uet_amr_description)/meshes/fl_caster_1.stl" scale="0.001 0.001 0.001"/>
+      <mesh filename="package://uet_amr_description/meshes/fl_caster_1.stl" scale="0.001 0.001 0.001"/>
     </geometry>
   </collision>
@@ -146,5 +146,5 @@
     <origin xyz="-0.218305 0.142031 0.065504" rpy="0 0 0"/>
     <geometry>
-      <mesh filename="file://$(find uet_amr_description)/meshes/fr_caster_1.stl" scale="0.001 0.001 0.001"/>
+      <mesh filename="package://uet_amr_description/meshes/fr_caster_1.stl" scale="0.001 0.001 0.001"/>
     </geometry>
     <material name="silver"/>
@@ -153,5 +153,5 @@
     <origin xyz="-0.218305 0.142031 0.065504" rpy="0 0 0"/>
     <geometry>
-      <mesh filename="file://$(find uet_amr_description)/meshes/fr_caster_1.stl" scale="0.001 0.001 0.001"/>
+      <mesh filename="package://uet_amr_description/meshes/fr_caster_1.stl" scale="0.001 0.001 0.001"/>
     </geometry>
   </collision>
@@ -166,5 +166,5 @@
     <origin xyz="-0.186479 -0.157654 0.117065" rpy="0 0 0"/>
     <geometry>
-      <mesh filename="file://$(find uet_amr_description)/meshes/fl_caster_wheel__1__1.stl" scale="0.001 0.001 0.001"/>
+      <mesh filename="package://uet_amr_description/meshes/fl_caster_wheel__1__1.stl" scale="0.001 0.001 0.001"/>
     </geometry>
     <material name="silver"/>
@@ -173,5 +173,5 @@
     <origin xyz="-0.186479 -0.157654 0.117065" rpy="0 0 0"/>
     <geometry>
-      <mesh filename="file://$(find uet_amr_description)/meshes/fl_caster_wheel__1__1.stl" scale="0.001 0.001 0.001"/>
+      <mesh filename="package://uet_amr_description/meshes/fl_caster_wheel__1__1.stl" scale="0.001 0.001 0.001"/>
     </geometry>
   </collision>
@@ -186,5 +186,5 @@
     <origin xyz="0.244519 -0.156443 0.117067" rpy="0 0 0"/>
     <geometry>
-      <mesh filename="file://$(find uet_amr_description)/meshes/bl_caster_wheel_1.stl" scale="0.001 0.001 0.001"/>
+      <mesh filename="package://uet_amr_description/meshes/bl_caster_wheel_1.stl" scale="0.001 0.001 0.001"/>
     </geometry>
     <material name="silver"/>
@@ -193,5 +193,5 @@
     <origin xyz="0.244519 -0.156443 0.117067" rpy="0 0 0"/>
     <geometry>
-      <mesh filename="file://$(find uet_amr_description)/meshes/bl_caster_wheel_1.stl" scale="0.001 0.001 0.001"/>
+      <mesh filename="package://uet_amr_description/meshes/bl_caster_wheel_1.stl" scale="0.001 0.001 0.001"/>
     </geometry>
   </collision>
@@ -206,5 +206,5 @@
     <origin xyz="0.243668 0.158053 0.118507" rpy="0 0 0"/>
     <geometry>
-      <mesh filename="file://$(find uet_amr_description)/meshes/br_caster_wheel_1.stl" scale="0.001 0.001 0.001"/>
+      <mesh filename="package://uet_amr_description/meshes/br_caster_wheel_1.stl" scale="0.001 0.001 0.001"/>
     </geometry>
     <material name="silver"/>
@@ -213,5 +213,5 @@
     <origin xyz="0.243668 0.158053 0.118507" rpy="0 0 0"/>
     <geometry>
-      <mesh filename="file://$(find uet_amr_description)/meshes/br_caster_wheel_1.stl" scale="0.001 0.001 0.001"/>
+      <mesh filename="package://uet_amr_description/meshes/br_caster_wheel_1.stl" scale="0.001 0.001 0.001"/>
     </geometry>
   </collision>
@@ -226,5 +226,5 @@
     <origin xyz="-0.18733 0.156841 0.118505" rpy="0 0 0"/>
     <geometry>
-      <mesh filename="file://$(find uet_amr_description)/meshes/fr_caster_wheel_1.stl" scale="0.001 0.001 0.001"/>
+      <mesh filename="package://uet_amr_description/meshes/fr_caster_wheel_1.stl" scale="0.001 0.001 0.001"/>
     </geometry>
     <material name="silver"/>
@@ -233,9 +233,9 @@
     <origin xyz="-0.18733 0.156841 0.118505" rpy="0 0 0"/>
     <geometry>
-      <mesh filename="file://$(find uet_amr_description)/meshes/fr_caster_wheel_1.stl" scale="0.001 0.001 0.001"/>
-    </geometry>
-  </collision>
-</link>
-<joint name="Revolute 17" type="continuous">
+      <mesh filename="package://uet_amr_description/meshes/fr_caster_wheel_1.stl" scale="0.001 0.001 0.001"/>
+    </geometry>
+  </collision>
+</link>
+<joint name="left_wheel_joint" type="continuous">
   <origin xyz="0.001978 0.151669 -0.077157" rpy="0 0 0"/>
   <parent link="base_link"/>
@@ -243,5 +243,5 @@
   <axis xyz="0 1 0"/>
 </joint>
-<joint name="Revolute 18" type="continuous">
+<joint name="right_wheel_joint" type="continuous">
   <origin xyz="0.002833 -0.152327 -0.078549" rpy="0 0 0"/>
   <parent link="base_link"/>
@@ -405,8 +405,8 @@
   <origin xyz="0.25 0.0 0.08" rpy="0 0 0"/>
 </joint>
-<link name="camera_depth_frame"></link>
+<link name="camera_depth_optical_frame"></link>
 <joint name="camera_depth_joint" type="fixed">
   <parent link="camera_link"/>
-  <child link="camera_depth_frame"/>
+  <child link="camera_depth_optical_frame"/>
   <origin xyz="0 0 0" rpy="-1.570796 0 -1.570796"/>
 </joint>

Commit message: chore: refactor, fix missing metadata, separated big robot into parts

File: ros2/src/uet_amr_description/urdf/materials.xacro (robot description, xacro)
@@ -1,6 +1,6 @@
 <?xml version="1.0" ?>
 <robot name="uet_amr" xmlns:xacro="http://www.ros.org/wiki/xacro" >
-<material name="silver">
-  <color rgba="0.700 0.700 0.700 1.000"/>
-</material>
+    <material name="silver">
+        <color rgba="0.700 0.700 0.700 1.000"/>
+    </material>
 </robot>

File: ros2/src/uet_amr_description/urdf/sensors/depth_camera.xacro (robot description, xacro)
@@ -1,88 +1,85 @@
 <?xml version="1.0"?>
 <robot xmlns:xacro="http://www.ros.org/wiki/xacro">
-  <xacro:macro name="depth_camera"
-               params="*origin parent update_rate horizontal_fov image_width image_height clip_near clip_far frame_id topic_name imu_update_rate imu_topic_name">
-    <link name="${frame_id}">
-      <visual>
-        <origin xyz="0 0 0" rpy="0 0 0"/>
-        <geometry>
-          <box size="0.025 0.065 0.025"/>
-        </geometry>
-        <material name="silver_cam">
-          <color rgba="0.75 0.75 0.75 1.0"/>
-        </material>
-      </visual>
-      <visual>
-        <origin xyz="0 -0.0325 0" rpy="0 0 0"/>
-        <geometry>
-          <cylinder length="0.025" radius="0.0125"/>
-        </geometry>
-        <material name="silver_cam"/>
-      </visual>
-      <visual>
-        <origin xyz="0 0.0325 0" rpy="0 0 0"/>
-        <geometry>
-          <cylinder length="0.025" radius="0.0125"/>
-        </geometry>
-        <material name="silver_cam"/>
-      </visual>
-      <collision>
-        <origin xyz="0 0 0" rpy="0 0 0"/>
-        <geometry>
-          <box size="0.025 0.090 0.025"/>
-        </geometry>
-      </collision>
-      <inertial>
-        <mass value="0.072"/>
-        <inertia ixx="0.00005" ixy="0.0" ixz="0.0"
-                 iyy="0.00001" iyz="0.0"
-                 izz="0.00005"/>
-      </inertial>
-    </link>
-    <joint name="${frame_id}_joint" type="fixed">
-      <parent link="${parent}"/>
-      <child  link="${frame_id}"/>
-      <xacro:insert_block name="origin"/>
-    </joint>
-    <link name="${frame_id}_optical"></link>
-    <joint name="${frame_id}_optical_joint" type="fixed">
-      <parent link="${frame_id}"/>
-      <child  link="${frame_id}_optical"/>
-      <origin xyz="0 0 0" rpy="-1.570796 0 -1.570796"/>
-    </joint>
-    <gazebo reference="${frame_id}">
-      <material>Gazebo/Red</material>
-      <sensor name="${frame_id}" type="rgbd_camera">
-        <pose>0 0 0 0 0 0</pose>
-        <visualize>true</visualize>
-        <update_rate>${update_rate}</update_rate>
-        <topic>${topic_name}</topic>
-        <ignition_frame_id>${frame_id}_optical</ignition_frame_id>
-        <camera>
-          <horizontal_fov>${horizontal_fov}</horizontal_fov>
-          <image>
-            <format>R8G8B8</format>
-            <width>${image_width}</width>
-            <height>${image_height}</height>
-          </image>
-          <clip>
-            <near>${clip_near}</near>
-            <far>${clip_far}</far>
-          </clip>
-          <noise>
-            <type>gaussian</type>
-            <mean>0.0</mean>
-            <stddev>0.007</stddev>
-          </noise>
-        </camera>
-      </sensor>
-      <sensor name="${frame_id}_imu" type="imu">
-        <always_on>true</always_on>
-        <update_rate>${imu_update_rate}</update_rate>
-        <visualize>false</visualize>
-        <topic>${imu_topic_name}</topic>
-        <ignition_frame_id>${frame_id}</ignition_frame_id>
-      </sensor>
-    </gazebo>
-  </xacro:macro>
+    <xacro:macro name="depth_camera" params="frame_id parent topic_name update_rate horizontal_fov image_width image_height clip_near clip_far imu_update_rate imu_topic_name *origin">
+        <link name="${frame_id}">
+            <visual>
+                <origin xyz="0 0 0" rpy="0 0 0"/>
+                <geometry>
+                    <box size="0.025 0.065 0.025"/>
+                </geometry>
+                <material name="silver_cam">
+                    <color rgba="0.75 0.75 0.75 1.0"/>
+                </material>
+            </visual>
+            <visual>
+                <origin xyz="0 -0.0325 0" rpy="0 0 0"/>
+                <geometry>
+                    <cylinder length="0.025" radius="0.0125"/>
+                </geometry>
+                <material name="silver_cam"/>
+            </visual>
+            <visual>
+                <origin xyz="0 0.0325 0" rpy="0 0 0"/>
+                <geometry>
+                    <cylinder length="0.025" radius="0.0125"/>
+                </geometry>
+                <material name="silver_cam"/>
+            </visual>
+            <collision>
+                <origin xyz="0 0 0" rpy="0 0 0"/>
+                <geometry>
+                    <box size="0.025 0.090 0.025"/>
+                </geometry>
+            </collision>
+            <inertial>
+                <mass value="0.072"/>
+                <inertia ixx="0.00005" ixy="0.0" ixz="0.0" iyy="0.00001" iyz="0.0" izz="0.00005"/>
+            </inertial>
+        </link>
+        <joint name="${frame_id}_joint" type="fixed">
+            <parent link="${parent}"/>
+            <child link="${frame_id}"/>
+            <xacro:insert_block name="origin"/>
+        </joint>
+        <link name="${frame_id}_optical"/>
+        <joint name="${frame_id}_optical_joint" type="fixed">
+            <parent link="${frame_id}"/>
+            <child link="${frame_id}_optical"/>
+            <origin xyz="0 0 0" rpy="-1.570796 0 -1.570796"/>
+        </joint>
+        <gazebo reference="${frame_id}">
+            <material>Gazebo/Red</material>
+            <sensor name="${frame_id}" type="rgbd_camera">
+                <pose>0 0 0 0 0 0</pose>
+                <visualize>true</visualize>
+                <update_rate>${update_rate}</update_rate>
+                <topic>${topic_name}</topic>
+                <ignition_frame_id>${frame_id}_optical</ignition_frame_id>
+                <camera>
+                    <horizontal_fov>${horizontal_fov}</horizontal_fov>
+                    <image>
+                        <format>R8G8B8</format>
+                        <width>${image_width}</width>
+                        <height>${image_height}</height>
+                    </image>
+                    <clip>
+                        <near>${clip_near}</near>
+                        <far>${clip_far}</far>
+                    </clip>
+                    <noise>
+                        <type>gaussian</type>
+                        <mean>0.0</mean>
+                        <stddev>0.007</stddev>
+                    </noise>
+                </camera>
+            </sensor>
+            <sensor name="${frame_id}_imu" type="imu">
+                <always_on>true</always_on>
+                <update_rate>${imu_update_rate}</update_rate>
+                <visualize>false</visualize>
+                <topic>${imu_topic_name}</topic>
+                <ignition_frame_id>${frame_id}</ignition_frame_id>
+            </sensor>
+        </gazebo>
+    </xacro:macro>
 </robot>

File: ros2/src/uet_amr_description/urdf/sensors/lidar.xacro (robot description, xacro)
@@ -1,54 +1,60 @@
 <?xml version="1.0"?>
 <robot xmlns:xacro="http://www.ros.org/wiki/xacro">
-  <xacro:macro name="lidar"
-               params="*origin parent update_rate ray_count min_angle max_angle min_range max_range frame_id topic_name">
-    <link name="${frame_id}">
-      <visual>
-        <geometry>
-          <cylinder length="0.04" radius="0.038"/>
-        </geometry>
-        <material name="blue">
-          <color rgba="0.0 0.4 0.8 1.0"/>
-        </material>
-      </visual>
-      <collision>
-        <geometry>
-          <cylinder length="0.04" radius="0.038"/>
-        </geometry>
-      </collision>
-      <inertial>
-        <mass value="0.185"/>
-        <inertia ixx="0.0001" ixy="0" ixz="0" iyy="0.0001" iyz="0" izz="0.0001"/>
-      </inertial>
-    </link>
-    <joint name="${frame_id}_joint" type="fixed">
-      <parent link="${parent}"/>
-      <child  link="${frame_id}"/>
-      <xacro:insert_block name="origin"/>
-    </joint>
-    <gazebo reference="${frame_id}">
-      <sensor name="${frame_id}" type="gpu_ray">
-        <always_on>true</always_on>
-        <visualize>true</visualize>
-        <update_rate>${update_rate}</update_rate>
-        <topic>${topic_name}</topic>
-        <ignition_frame_id>${frame_id}</ignition_frame_id>
-        <ray>
-          <scan>
-            <horizontal>
-              <samples>${ray_count}</samples>
-              <resolution>1</resolution>
-              <min_angle>${min_angle}</min_angle>
-              <max_angle>${max_angle}</max_angle>
-            </horizontal>
-          </scan>
-          <range>
-            <min>${min_range}</min>
-            <max>${max_range}</max>
-            <resolution>0.001</resolution>
-          </range>
-        </ray>
-      </sensor>
-    </gazebo>
-  </xacro:macro>
+    <xacro:macro name="lidar" params="frame_id parent topic_name update_rate ray_count min_angle max_angle min_range max_range *origin">
+        <link name="${frame_id}">
+            <visual>
+                <geometry>
+                    <cylinder length="0.04" radius="0.038"/>
+                </geometry>
+                <material name="blue">
+                    <color rgba="0.0 0.4 0.8 1.0"/>
+                </material>
+            </visual>
+            <collision>
+                <geometry>
+                    <cylinder length="0.04" radius="0.038"/>
+                </geometry>
+            </collision>
+            <inertial>
+                <mass value="0.185"/>
+                <inertia ixx="0.0000914" ixy="0" ixz="0" iyy="0.0000914" iyz="0" izz="0.0001335"/>
+            </inertial>
+        </link>
+        <joint name="${frame_id}_joint" type="fixed">
+            <parent link="${parent}"/>
+            <child link="${frame_id}"/>
+            <xacro:insert_block name="origin"/>
+        </joint>
+        <gazebo reference="${frame_id}">
+            <visual>
+                <material>
+                    <ambient>0.0 0.4 0.8 1.0</ambient>
+                    <diffuse>0.0 0.4 0.8 1.0</diffuse>
+                    <specular>0.1 0.1 0.1 1.0</specular>
+                </material>
+            </visual>
+            <sensor name="${frame_id}" type="gpu_lidar">
+                <always_on>true</always_on>
+                <visualize>true</visualize>
+                <update_rate>${update_rate}</update_rate>
+                <topic>${topic_name}</topic>
+                <ignition_frame_id>${frame_id}</ignition_frame_id>
+                <lidar>
+                    <scan>
+                        <horizontal>
+                            <samples>${ray_count}</samples>
+                            <resolution>1</resolution>
+                            <min_angle>${min_angle}</min_angle>
+                            <max_angle>${max_angle}</max_angle>
+                        </horizontal>
+                    </scan>
+                    <range>
+                        <min>${min_range}</min>
+                        <max>${max_range}</max>
+                        <resolution>0.001</resolution>
+                    </range>
+                </lidar>
+            </sensor>
+        </gazebo>
+    </xacro:macro>
 </robot>
