Commit message: change gazebo version from classic to fortress and add controller config for robot

File: ros2/src/uet_amr_description/urdf/uet_amr.xacro (robot description, xacro)
@@ -2,14 +2,14 @@
 <robot name="uet_amr" xmlns:xacro="http://www.ros.org/wiki/xacro">
 <xacro:include filename="$(find uet_amr_description)/urdf/materials.xacro" />
-<xacro:include filename="$(find uet_amr_description)/urdf/uet_amr.trans" />
+<xacro:include filename="$(find uet_amr_description)/urdf/uet_amr.ros2control" />
 <xacro:include filename="$(find uet_amr_description)/urdf/uet_amr.gazebo" />
 <link name="base_link">
   <inertial>
-    <origin xyz="0.00090860894185851 -9.962260545167594e-05 0.15815402081981028" rpy="0 0 0"/>
+    <origin xyz="0.00090860894185851 -9.962260545167594e-05 0.00815402081981028" rpy="0 0 0"/>
     <mass value="9.278155760715826"/>
     <inertia ixx="0.375602" iyy="0.23114" izz="0.56136" ixy="0.000644" iyz="0.000485" ixz="-0.001482"/>
   </inertial>
   <visual>
-    <origin xyz="0 0 0" rpy="0 0 0"/>
+    <origin xyz="0 0 -0.15" rpy="0 0 0"/>
     <geometry>
       <mesh filename="file://$(find uet_amr_description)/meshes/base_link.stl" scale="0.001 0.001 0.001"/>
@@ -18,5 +18,5 @@
   </visual>
   <collision>
-    <origin xyz="0 0 0" rpy="0 0 0"/>
+    <origin xyz="0 0 -0.15" rpy="0 0 0"/>
     <geometry>
       <mesh filename="file://$(find uet_amr_description)/meshes/base_link.stl" scale="0.001 0.001 0.001"/>
@@ -225,17 +225,17 @@
 </link>
 <joint name="Revolute 17" type="continuous">
-  <origin xyz="0.151679 0.000357 0.088358" rpy="0 0 0"/>
+  <origin xyz="0.151679 0.000357 -0.061642" rpy="0 0 0"/>
   <parent link="base_link"/>
   <child link="left_wheel_1"/>
-  <axis xyz="0.999992 0.00281 0.002891"/>
+  <axis xyz="-1 0 0"/>
 </joint>
 <joint name="Revolute 18" type="continuous">
-  <origin xyz="-0.152318 -0.000498 0.08748" rpy="0 0 0"/>
+  <origin xyz="-0.152318 -0.000498 -0.06252" rpy="0 0 0"/>
   <parent link="base_link"/>
   <child link="right_wheel_1"/>
-  <axis xyz="-0.999992 -0.00281 -0.002891"/>
+  <axis xyz="-1 0 0"/>
 </joint>
 <joint name="Revolute 19" type="continuous">
-  <origin xyz="0.141287 0.21585 0.100966" rpy="0 0 0"/>
+  <origin xyz="0.141287 0.21585 -0.049034" rpy="0 0 0"/>
   <parent link="base_link"/>
   <child link="bl_caster_1"/>
@@ -249,5 +249,5 @@
 </joint>
 <joint name="Revolute 21" type="continuous">
-  <origin xyz="-0.143211 0.21505 0.100144" rpy="0 0 0"/>
+  <origin xyz="-0.143211 0.21505 -0.049856" rpy="0 0 0"/>
   <parent link="base_link"/>
   <child link="br_caster_1"/>
@@ -261,5 +261,5 @@
 </joint>
 <joint name="Revolute 23" type="continuous">
-  <origin xyz="0.142496 -0.215148 0.101694" rpy="0 0 0"/>
+  <origin xyz="0.142496 -0.215148 -0.048306" rpy="0 0 0"/>
   <parent link="base_link"/>
   <child link="fl_caster_1"/>
@@ -273,5 +273,5 @@
 </joint>
 <joint name="Revolute 25" type="continuous">
-  <origin xyz="-0.142002 -0.215947 0.100872" rpy="0 0 0"/>
+  <origin xyz="-0.142002 -0.215947 -0.049128" rpy="0 0 0"/>
   <parent link="base_link"/>
   <child link="fr_caster_1"/>
@@ -306,5 +306,5 @@
   <parent link="base_link"/>
   <child  link="lidar_link_1"/>
-  <origin xyz="0.15 0.23 0.255" rpy="0 0 0"/>
+  <origin xyz="0.15 0.23 0.105" rpy="0 0 0"/>
 </joint>
 <!-- <link name="lidar_link_2">
@@ -330,5 +330,5 @@
   <parent link="base_link"/>
   <child link="lidar_link_2"/>
-  <origin xyz="-0.15 -0.23 0.255" rpy="0 0 3.14159"/>
+  <origin xyz="-0.15 -0.23 0.105" rpy="0 0 3.14159"/>
 </joint> -->
 <link name="imu_link">
@@ -348,5 +348,5 @@
   <parent link="base_link"/>
   <child  link="imu_link"/>
-  <origin xyz="0.02 0.255 0.246" rpy="0 0 0"/>
+  <origin xyz="0.02 0.255 0.096" rpy="0 0 0"/>
 </joint>
 <link name="camera_link">
@@ -390,5 +390,5 @@
   <parent link="base_link"/>
   <child link="camera_link"/>
-  <origin xyz="0.0 0.25 0.246" rpy="0 0 1.570796"/>
+  <origin xyz="0.0 0.25 0.096" rpy="0 0 1.570796"/>
 </joint>
 <link name="camera_depth_frame"></link>

Commit message: add-basefootprint-for-urdf

File: ros2/src/uet_amr_description/urdf/uet_amr.xacro (robot description, xacro)
@@ -24,4 +24,12 @@
   </collision>
 </link>
+    <!-- BASE_FOOTPRINT LINK -->
+    <joint name="base_footprint_joint" type="fixed">
+        <parent link="base_link"/>
+        <child link="base_footprint"/>
+        <origin xyz="0 0 0" rpy="0 0 0"/>
+    </joint>
+    <link name="base_footprint">
+    </link>
 <link name="left_wheel_1">
   <inertial>

Commit message: update

File: ros2/src/uet_amr_description/urdf/uet_amr.xacro (robot description, xacro)
@@ -24,12 +24,11 @@
   </collision>
 </link>
-    <!-- BASE_FOOTPRINT LINK -->
-    <joint name="base_footprint_joint" type="fixed">
-        <parent link="base_link"/>
-        <child link="base_footprint"/>
-        <origin xyz="0 0 0" rpy="0 0 0"/>
-    </joint>
-    <link name="base_footprint">
-    </link>
+<joint name="base_footprint_joint" type="fixed">
+    <parent link="base_link"/>
+    <child link="base_footprint"/>
+    <origin xyz="0 0 0" rpy="0 0 0"/>
+</joint>
+<link name="base_footprint">
+</link>
 <link name="left_wheel_1">
   <inertial>

Commit message: update urdf files

File: ros2/src/uet_amr_description/urdf/uet_amr.xacro (robot description, xacro)
@@ -12,10 +12,10 @@
 <link name="base_link">
   <inertial>
-    <origin xyz="0.00090860894185851 -9.962260545167594e-05 0.00815402081981028" rpy="0 0 0"/>
-    <mass value="9.278155760715826"/>
-    <inertia ixx="0.375602" iyy="0.23114" izz="0.56136" ixy="0.000644" iyz="0.000485" ixz="-0.001482"/>
-  </inertial>
-  <visual>
-    <origin xyz="0 0 -0.15" rpy="0 0 0"/>
+    <origin xyz="0.0025532775935351716 0.0007810393984697188 -0.007616605165089496" rpy="0 0 0"/>
+    <mass value="9.278155762193999"/>
+    <inertia ixx="0.231139" iyy="0.375607" izz="0.561355" ixy="-0.000648" iyz="-0.001793" ixz="7.2e-05"/>
+  </inertial>
+  <visual>
+    <origin xyz="0 0 0" rpy="0 0 0"/>
     <geometry>
       <mesh filename="file://$(find uet_amr_description)/meshes/base_link.stl" scale="0.001 0.001 0.001"/>
@@ -24,5 +24,5 @@
   </visual>
   <collision>
-    <origin xyz="0 0 -0.15" rpy="0 0 0"/>
+    <origin xyz="0 0 0" rpy="0 0 0"/>
     <geometry>
       <mesh filename="file://$(find uet_amr_description)/meshes/base_link.stl" scale="0.001 0.001 0.001"/>
@@ -39,10 +39,10 @@
 <link name="left_wheel_1">
   <inertial>
-    <origin xyz="0.06626336710358052 0.000190571908891459 0.0001966883827906052" rpy="0 0 0"/>
-    <mass value="8.133164726083537"/>
-    <inertia ixx="0.026227" iyy="0.014975" izz="0.014975" ixy="3.4e-05" iyz="0.0" ixz="3.5e-05"/>
-  </inertial>
-  <visual>
-    <origin xyz="-0.151679 -0.000357 -0.088358" rpy="0 0 0"/>
+    <origin xyz="-0.0001975256393499439 0.06876256340886683 0.0003191159733880039" rpy="0 0 0"/>
+    <mass value="8.133156223625377"/>
+    <inertia ixx="0.014975" iyy="0.026227" izz="0.014975" ixy="-3.4e-05" iyz="5.4e-05" ixz="-0.0"/>
+  </inertial>
+  <visual>
+    <origin xyz="-0.001978 -0.151669 0.077157" rpy="0 0 0"/>
     <geometry>
       <mesh filename="file://$(find uet_amr_description)/meshes/left_wheel_1.stl" scale="0.001 0.001 0.001"/>
@@ -51,5 +51,5 @@
   </visual>
   <collision>
-    <origin xyz="-0.151679 -0.000357 -0.088358" rpy="0 0 0"/>
+    <origin xyz="-0.001978 -0.151669 0.077157" rpy="0 0 0"/>
     <geometry>
       <mesh filename="file://$(find uet_amr_description)/meshes/left_wheel_1.stl" scale="0.001 0.001 0.001"/>
@@ -59,10 +59,10 @@
 <link name="right_wheel_1">
   <inertial>
-    <origin xyz="-0.06626360584895855 -0.00017973253869872944 -0.000188979602087469" rpy="0 0 0"/>
-    <mass value="8.1331638221686"/>
-    <inertia ixx="0.026227" iyy="0.014975" izz="0.014975" ixy="2.9e-05" iyz="0.0" ixz="3.1e-05"/>
-  </inertial>
-  <visual>
-    <origin xyz="0.152318 0.000498 -0.08748" rpy="0 0 0"/>
+    <origin xyz="0.00018681806470619271 -0.06876255933824524 -0.00031221526229738283" rpy="0 0 0"/>
+    <mass value="8.133163359417004"/>
+    <inertia ixx="0.014975" iyy="0.026227" izz="0.014975" ixy="-2.9e-05" iyz="5e-05" ixz="-0.0"/>
+  </inertial>
+  <visual>
+    <origin xyz="-0.002833 0.152327 0.078549" rpy="0 0 0"/>
     <geometry>
       <mesh filename="file://$(find uet_amr_description)/meshes/right_wheel_1.stl" scale="0.001 0.001 0.001"/>
@@ -71,5 +71,5 @@
   </visual>
   <collision>
-    <origin xyz="0.152318 0.000498 -0.08748" rpy="0 0 0"/>
+    <origin xyz="-0.002833 0.152327 0.078549" rpy="0 0 0"/>
     <geometry>
       <mesh filename="file://$(find uet_amr_description)/meshes/right_wheel_1.stl" scale="0.001 0.001 0.001"/>
@@ -79,10 +79,10 @@
 <link name="bl_caster_1">
   <inertial>
-    <origin xyz="-0.00010040633192423543 0.016286651357198645 -0.022951903402420232" rpy="0 0 0"/>
-    <mass value="0.13840813854724046"/>
-    <inertia ixx="0.00011" iyy="0.000106" izz="6.3e-05" ixy="0.0" iyz="3.3e-05" ixz="-0.0"/>
-  </inertial>
-  <visual>
-    <origin xyz="-0.141287 -0.21585 -0.100966" rpy="0 0 0"/>
+    <origin xyz="-0.016325683724505796 -6.209736988929682e-05 -0.02292504256915545" rpy="0 0 0"/>
+    <mass value="0.1384081385472382"/>
+    <inertia ixx="0.000106" iyy="0.00011" izz="6.3e-05" ixy="-0.0" iyz="-0.0" ixz="-3.3e-05"/>
+  </inertial>
+  <visual>
+    <origin xyz="0.213493 -0.141254 0.064203" rpy="0 0 0"/>
     <geometry>
       <mesh filename="file://$(find uet_amr_description)/meshes/bl_caster_1.stl" scale="0.001 0.001 0.001"/>
@@ -91,5 +91,5 @@
   </visual>
   <collision>
-    <origin xyz="-0.141287 -0.21585 -0.100966" rpy="0 0 0"/>
+    <origin xyz="0.213493 -0.141254 0.064203" rpy="0 0 0"/>
     <geometry>
       <mesh filename="file://$(find uet_amr_description)/meshes/bl_caster_1.stl" scale="0.001 0.001 0.001"/>
@@ -97,12 +97,92 @@
   </collision>
 </link>
+<link name="br_caster_1">
+  <inertial>
+    <origin xyz="-0.016325165192457858 -6.199154591685074e-05 -0.02292460400344691" rpy="0 0 0"/>
+    <mass value="0.13840813854723946"/>
+    <inertia ixx="0.000106" iyy="0.00011" izz="6.3e-05" ixy="-0.0" iyz="-0.0" ixz="-3.3e-05"/>
+  </inertial>
+  <visual>
+    <origin xyz="0.212694 0.143242 0.065506" rpy="0 0 0"/>
+    <geometry>
+      <mesh filename="file://$(find uet_amr_description)/meshes/br_caster_1.stl" scale="0.001 0.001 0.001"/>
+    </geometry>
+    <material name="silver"/>
+  </visual>
+  <collision>
+    <origin xyz="0.212694 0.143242 0.065506" rpy="0 0 0"/>
+    <geometry>
+      <mesh filename="file://$(find uet_amr_description)/meshes/br_caster_1.stl" scale="0.001 0.001 0.001"/>
+    </geometry>
+  </collision>
+</link>
+<link name="fl_caster_1">
+  <inertial>
+    <origin xyz="-0.01632538566149161 -6.187397013268647e-05 -0.022924882170905936" rpy="0 0 0"/>
+    <mass value="0.13840813854723621"/>
+    <inertia ixx="0.000106" iyy="0.00011" izz="6.3e-05" ixy="-0.0" iyz="-0.0" ixz="-3.3e-05"/>
+  </inertial>
+  <visual>
+    <origin xyz="-0.217505 -0.142465 0.064201" rpy="0 0 0"/>
+    <geometry>
+      <mesh filename="file://$(find uet_amr_description)/meshes/fl_caster_1.stl" scale="0.001 0.001 0.001"/>
+    </geometry>
+    <material name="silver"/>
+  </visual>
+  <collision>
+    <origin xyz="-0.217505 -0.142465 0.064201" rpy="0 0 0"/>
+    <geometry>
+      <mesh filename="file://$(find uet_amr_description)/meshes/fl_caster_1.stl" scale="0.001 0.001 0.001"/>
+    </geometry>
+  </collision>
+</link>
+<link name="fr_caster_1">
+  <inertial>
+    <origin xyz="-0.016325867129421662 -6.17681461664299e-05 -0.022924443605240485" rpy="0 0 0"/>
+    <mass value="0.13840813854723868"/>
+    <inertia ixx="0.000106" iyy="0.00011" izz="6.3e-05" ixy="-0.0" iyz="-0.0" ixz="-3.3e-05"/>
+  </inertial>
+  <visual>
+    <origin xyz="-0.218305 0.142031 0.065504" rpy="0 0 0"/>
+    <geometry>
+      <mesh filename="file://$(find uet_amr_description)/meshes/fr_caster_1.stl" scale="0.001 0.001 0.001"/>
+    </geometry>
+    <material name="silver"/>
+  </visual>
+  <collision>
+    <origin xyz="-0.218305 0.142031 0.065504" rpy="0 0 0"/>
+    <geometry>
+      <mesh filename="file://$(find uet_amr_description)/meshes/fr_caster_1.stl" scale="0.001 0.001 0.001"/>
+    </geometry>
+  </collision>
+</link>
+<link name="fl_caster_wheel__1__1">
+  <inertial>
+    <origin xyz="2.5615176473869905e-05 -0.014999755176358459 -6.848949303683849e-05" rpy="0 0 0"/>
+    <mass value="0.9168727321007171"/>
+    <inertia ixx="0.000422" iyy="0.000731" izz="0.000422" ixy="-1e-06" iyz="1e-06" ixz="-0.0"/>
+  </inertial>
+  <visual>
+    <origin xyz="-0.186479 -0.157654 0.117065" rpy="0 0 0"/>
+    <geometry>
+      <mesh filename="file://$(find uet_amr_description)/meshes/fl_caster_wheel__1__1.stl" scale="0.001 0.001 0.001"/>
+    </geometry>
+    <material name="silver"/>
+  </visual>
+  <collision>
+    <origin xyz="-0.186479 -0.157654 0.117065" rpy="0 0 0"/>
+    <geometry>
+      <mesh filename="file://$(find uet_amr_description)/meshes/fl_caster_wheel__1__1.stl" scale="0.001 0.001 0.001"/>
+    </geometry>
+  </collision>
+</link>
 <link name="bl_caster_wheel_1">
   <inertial>
-    <origin xyz="-0.014999717472892915 -2.604639410183629e-05 -4.362998470474472e-05" rpy="0 0 0"/>
-    <mass value="0.9168727321007148"/>
-    <inertia ixx="0.000731" iyy="0.000422" izz="0.000422" ixy="1e-06" iyz="0.0" ixz="1e-06"/>
-  </inertial>
-  <visual>
-    <origin xyz="-0.156387 -0.246787 -0.048025" rpy="0 0 0"/>
+    <origin xyz="2.531711346762111e-05 -0.01499997857611493 -6.864989128550769e-05" rpy="0 0 0"/>
+    <mass value="0.9168727321007182"/>
+    <inertia ixx="0.000422" iyy="0.000731" izz="0.000422" ixy="-1e-06" iyz="1e-06" ixz="-0.0"/>
+  </inertial>
+  <visual>
+    <origin xyz="0.244519 -0.156443 0.117067" rpy="0 0 0"/>
     <geometry>
       <mesh filename="file://$(find uet_amr_description)/meshes/bl_caster_wheel_1.stl" scale="0.001 0.001 0.001"/>
@@ -111,5 +191,5 @@
   </visual>
   <collision>
-    <origin xyz="-0.156387 -0.246787 -0.048025" rpy="0 0 0"/>
+    <origin xyz="0.244519 -0.156443 0.117067" rpy="0 0 0"/>
     <geometry>
       <mesh filename="file://$(find uet_amr_description)/meshes/bl_caster_wheel_1.stl" scale="0.001 0.001 0.001"/>
@@ -117,32 +197,12 @@
   </collision>
 </link>
-<link name="br_caster_1">
-  <inertial>
-    <origin xyz="-0.00010009418282455607 0.016287130720061577 -0.022952323166481686" rpy="0 0 0"/>
-    <mass value="0.1384081385472399"/>
-    <inertia ixx="0.00011" iyy="0.000106" izz="6.3e-05" ixy="0.0" iyz="3.3e-05" ixz="-0.0"/>
-  </inertial>
-  <visual>
-    <origin xyz="0.143211 -0.21505 -0.100144" rpy="0 0 0"/>
-    <geometry>
-      <mesh filename="file://$(find uet_amr_description)/meshes/br_caster_1.stl" scale="0.001 0.001 0.001"/>
-    </geometry>
-    <material name="silver"/>
-  </visual>
-  <collision>
-    <origin xyz="0.143211 -0.21505 -0.100144" rpy="0 0 0"/>
-    <geometry>
-      <mesh filename="file://$(find uet_amr_description)/meshes/br_caster_1.stl" scale="0.001 0.001 0.001"/>
-    </geometry>
-  </collision>
-</link>
 <link name="br_caster_wheel_1">
   <inertial>
-    <origin xyz="0.014999594676208011 2.543296876336698e-05 4.2950251234505354e-05" rpy="0 0 0"/>
-    <mass value="0.9168727321007151"/>
-    <inertia ixx="0.000731" iyy="0.000422" izz="0.000422" ixy="1e-06" iyz="0.0" ixz="1e-06"/>
-  </inertial>
-  <visual>
-    <origin xyz="0.15811 -0.245936 -0.047116" rpy="0 0 0"/>
+    <origin xyz="-2.6164354486490904e-05 0.015000127247860873 6.878867442251801e-05" rpy="0 0 0"/>
+    <mass value="0.9168727321007177"/>
+    <inertia ixx="0.000422" iyy="0.000731" izz="0.000422" ixy="-1e-06" iyz="1e-06" ixz="-0.0"/>
+  </inertial>
+  <visual>
+    <origin xyz="0.243668 0.158053 0.118507" rpy="0 0 0"/>
     <geometry>
       <mesh filename="file://$(find uet_amr_description)/meshes/br_caster_wheel_1.stl" scale="0.001 0.001 0.001"/>
@@ -151,5 +211,5 @@
   </visual>
   <collision>
-    <origin xyz="0.15811 -0.245936 -0.047116" rpy="0 0 0"/>
+    <origin xyz="0.243668 0.158053 0.118507" rpy="0 0 0"/>
     <geometry>
       <mesh filename="file://$(find uet_amr_description)/meshes/br_caster_wheel_1.stl" scale="0.001 0.001 0.001"/>
@@ -157,72 +217,12 @@
   </collision>
 </link>
-<link name="fl_caster_1">
-  <inertial>
-    <origin xyz="-0.00010028275687246069 0.016286962152481682 -0.022951947100197004" rpy="0 0 0"/>
-    <mass value="0.1384081385472415"/>
-    <inertia ixx="0.00011" iyy="0.000106" izz="6.3e-05" ixy="0.0" iyz="3.3e-05" ixz="-0.0"/>
-  </inertial>
-  <visual>
-    <origin xyz="-0.142496 0.215148 -0.101694" rpy="0 0 0"/>
-    <geometry>
-      <mesh filename="file://$(find uet_amr_description)/meshes/fl_caster_1.stl" scale="0.001 0.001 0.001"/>
-    </geometry>
-    <material name="silver"/>
-  </visual>
-  <collision>
-    <origin xyz="-0.142496 0.215148 -0.101694" rpy="0 0 0"/>
-    <geometry>
-      <mesh filename="file://$(find uet_amr_description)/meshes/fl_caster_1.stl" scale="0.001 0.001 0.001"/>
-    </geometry>
-  </collision>
-</link>
-<link name="fl_caster_wheel__1__1">
-  <inertial>
-    <origin xyz="-0.01499959389784103 -2.573559881430265e-05 -4.3673682482696374e-05" rpy="0 0 0"/>
-    <mass value="0.9168727321007141"/>
-    <inertia ixx="0.000731" iyy="0.000422" izz="0.000422" ixy="1e-06" iyz="0.0" ixz="1e-06"/>
-  </inertial>
-  <visual>
-    <origin xyz="-0.157596 0.184211 -0.048753" rpy="0 0 0"/>
-    <geometry>
-      <mesh filename="file://$(find uet_amr_description)/meshes/fl_caster_wheel__1__1.stl" scale="0.001 0.001 0.001"/>
-    </geometry>
-    <material name="silver"/>
-  </visual>
-  <collision>
-    <origin xyz="-0.157596 0.184211 -0.048753" rpy="0 0 0"/>
-    <geometry>
-      <mesh filename="file://$(find uet_amr_description)/meshes/fl_caster_wheel__1__1.stl" scale="0.001 0.001 0.001"/>
-    </geometry>
-  </collision>
-</link>
-<link name="fr_caster_1">
-  <inertial>
-    <origin xyz="-9.997060777847122e-05 0.01628644151532263 -0.022952366864301507" rpy="0 0 0"/>
-    <mass value="0.13840813854724168"/>
-    <inertia ixx="0.00011" iyy="0.000106" izz="6.3e-05" ixy="0.0" iyz="3.3e-05" ixz="-0.0"/>
-  </inertial>
-  <visual>
-    <origin xyz="0.142002 0.215947 -0.100872" rpy="0 0 0"/>
-    <geometry>
-      <mesh filename="file://$(find uet_amr_description)/meshes/fr_caster_1.stl" scale="0.001 0.001 0.001"/>
-    </geometry>
-    <material name="silver"/>
-  </visual>
-  <collision>
-    <origin xyz="0.142002 0.215947 -0.100872" rpy="0 0 0"/>
-    <geometry>
-      <mesh filename="file://$(find uet_amr_description)/meshes/fr_caster_1.stl" scale="0.001 0.001 0.001"/>
-    </geometry>
-  </collision>
-</link>
 <link name="fr_caster_wheel_1">
   <inertial>
-    <origin xyz="0.014999718251254152 2.574376402461609e-05 4.290655341319255e-05" rpy="0 0 0"/>
-    <mass value="0.9168727321007145"/>
-    <inertia ixx="0.000731" iyy="0.000422" izz="0.000422" ixy="1e-06" iyz="0.0" ixz="1e-06"/>
-  </inertial>
-  <visual>
-    <origin xyz="0.156901 0.185062 -0.047844" rpy="0 0 0"/>
+    <origin xyz="-2.586629145395758e-05 0.014999350647611681 6.894907262748606e-05" rpy="0 0 0"/>
+    <mass value="0.9168727321007173"/>
+    <inertia ixx="0.000422" iyy="0.000731" izz="0.000422" ixy="-1e-06" iyz="1e-06" ixz="-0.0"/>
+  </inertial>
+  <visual>
+    <origin xyz="-0.18733 0.156841 0.118505" rpy="0 0 0"/>
     <geometry>
       <mesh filename="file://$(find uet_amr_description)/meshes/fr_caster_wheel_1.stl" scale="0.001 0.001 0.001"/>
@@ -231,5 +231,5 @@
   </visual>
   <collision>
-    <origin xyz="0.156901 0.185062 -0.047844" rpy="0 0 0"/>
+    <origin xyz="-0.18733 0.156841 0.118505" rpy="0 0 0"/>
     <geometry>
       <mesh filename="file://$(find uet_amr_description)/meshes/fr_caster_wheel_1.stl" scale="0.001 0.001 0.001"/>
@@ -238,62 +238,62 @@
 </link>
 <joint name="Revolute 17" type="continuous">
-  <origin xyz="0.151679 0.000357 -0.061642" rpy="0 0 0"/>
+  <origin xyz="0.001978 0.151669 -0.077157" rpy="0 0 0"/>
   <parent link="base_link"/>
   <child link="left_wheel_1"/>
-  <axis xyz="-1 0 0"/>
+  <axis xyz="0 1 0"/>
 </joint>
 <joint name="Revolute 18" type="continuous">
-  <origin xyz="-0.152318 -0.000498 -0.06252" rpy="0 0 0"/>
+  <origin xyz="0.002833 -0.152327 -0.078549" rpy="0 0 0"/>
   <parent link="base_link"/>
   <child link="right_wheel_1"/>
-  <axis xyz="-1 0 0"/>
+  <axis xyz="0 1 0"/>
 </joint>
 <joint name="Revolute 19" type="continuous">
-  <origin xyz="0.141287 0.21585 -0.049034" rpy="0 0 0"/>
+  <origin xyz="-0.213493 0.141254 -0.064203" rpy="0 0 0"/>
   <parent link="base_link"/>
   <child link="bl_caster_1"/>
-  <axis xyz="0.002895 -0.001681 -0.999994"/>
+  <axis xyz="-8e-06 0.004578 -0.99999"/>
 </joint>
 <joint name="Revolute 20" type="continuous">
-  <origin xyz="0.0151 0.030937 -0.052941" rpy="0 0 0"/>
+  <origin xyz="-0.212694 -0.143242 -0.065506" rpy="0 0 0"/>
+  <parent link="base_link"/>
+  <child link="br_caster_1"/>
+  <axis xyz="-8e-06 0.004578 -0.99999"/>
+</joint>
+<joint name="Revolute 21" type="continuous">
+  <origin xyz="0.217505 0.142465 -0.064201" rpy="0 0 0"/>
+  <parent link="base_link"/>
+  <child link="fl_caster_1"/>
+  <axis xyz="-8e-06 0.004578 -0.99999"/>
+</joint>
+<joint name="Revolute 22" type="continuous">
+  <origin xyz="0.218305 -0.142031 -0.065504" rpy="0 0 0"/>
+  <parent link="base_link"/>
+  <child link="fr_caster_1"/>
+  <axis xyz="-8e-06 0.004578 -0.99999"/>
+</joint>
+<joint name="Revolute 23" type="continuous">
+  <origin xyz="-0.031026 0.015189 -0.052864" rpy="0 0 0"/>
+  <parent link="fl_caster_1"/>
+  <child link="fl_caster_wheel__1__1"/>
+  <axis xyz="0.001715 -0.999988 -0.004578"/>
+</joint>
+<joint name="Revolute 24" type="continuous">
+  <origin xyz="-0.031026 0.015189 -0.052864" rpy="0 0 0"/>
   <parent link="bl_caster_1"/>
   <child link="bl_caster_wheel_1"/>
-  <axis xyz="-0.999994 -0.001715 -0.002893"/>
-</joint>
-<joint name="Revolute 21" type="continuous">
-  <origin xyz="-0.143211 0.21505 -0.049856" rpy="0 0 0"/>
-  <parent link="base_link"/>
-  <child link="br_caster_1"/>
-  <axis xyz="0.002895 -0.001681 -0.999994"/>
-</joint>
-<joint name="Revolute 22" type="continuous">
-  <origin xyz="-0.014899 0.030886 -0.053028" rpy="0 0 0"/>
+  <axis xyz="0.001715 -0.999988 -0.004578"/>
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