Commit message: fix rviz2 lazer scan

File: ros2/src/uet_amr_description/urdf/uet_amr.xacro (robot description, xacro)
@@ -3,4 +3,6 @@
 <xacro:arg name="use_real_hardware" default="false"/>
 <xacro:include filename="$(find uet_amr_description)/urdf/materials.xacro" />
+<xacro:include filename="$(find uet_amr_description)/urdf/sensors/lidar.xacro" />
+<xacro:include filename="$(find uet_amr_description)/urdf/sensors/depth_camera.xacro" />
 <xacro:if value="$(arg use_real_hardware)">
   <xacro:include filename="$(find uet_amr_description)/urdf/uet_amr_real.ros2control" />
@@ -31,6 +33,6 @@
 </link>
 <joint name="base_footprint_joint" type="fixed">
-    <parent link="base_link"/>
-    <child link="base_footprint"/>
+    <parent link="base_footprint"/>
+    <child link="base_link"/>
     <origin xyz="0 0 0" rpy="0 0 0"/>
 </joint>
@@ -297,5 +299,16 @@
   <axis xyz="0.001715 -0.999988 -0.004578"/>
 </joint>
-<link name="lidar_link_1">
+<xacro:lidar parent="base_link"
+             update_rate="15"
+             ray_count="800"
+             min_angle="-3.14159"
+             max_angle="3.14159"
+             min_range="0.15"
+             max_range="25.0"
+             frame_id="laser"
+             topic_name="scan">
+  <origin xyz="0.25 -0.16 0.088" rpy="0 0 0"/>
+</xacro:lidar>
+<!-- <link name="lidar_link_2">
   <visual>
     <geometry>
@@ -313,28 +326,4 @@
   <inertial>
     <mass value="0.185"/>
-    <inertia ixx="0.0001" ixy="0" ixz="0" iyy="0.0001" iyz="0" izz="0.0001"/>
-  </inertial>
-</link>
-<joint name="lidar_joint" type="fixed">
-  <parent link="base_link"/>
-  <child  link="lidar_link_1"/>
-  <origin xyz="0.25 -0.16 0.088" rpy="0 0 0"/>
-</joint>
-<!-- <link name="lidar_link_2">
-  <visual>
-    <geometry>
-      <cylinder length="0.04" radius="0.038"/>
-    </geometry>
-    <material name="blue">
-      <color rgba="0.0 0.4 0.8 1.0"/>
-    </material>
-  </visual>
-  <collision>
-    <geometry>
-      <cylinder length="0.04" radius="0.038"/>
-    </geometry>
-  </collision>
-  <inertial>
-    <mass value="0.185"/>
     <inertia ixx="0.0001" ixy="0.0" ixz="0.0" iyy="0.0001" iyz="0.0" izz="0.0001"/>
   </inertial>
@@ -345,69 +334,16 @@
   <origin xyz="-0.15 -0.23 0.105" rpy="0 0 3.14159"/>
 </joint> -->
-<link name="imu_link">
-  <visual>
-    <geometry>
-      <box size="0.02 0.02 0.01"/>
-    </geometry>
-  </visual>
-  <inertial>
-    <mass value="0.01"/>
-    <inertia ixx="0.000001" ixy="0" ixz="0"
-              iyy="0.000001" iyz="0"
-              izz="0.000001"/>
-  </inertial>
-</link>
-<joint name="imu_joint" type="fixed">
-  <parent link="base_link"/>
-  <child  link="imu_link"/>
-  <origin xyz="0.26 -0.02 0.085" rpy="0 0 0"/>
-</joint>
-<link name="camera_link">
-<visual>
-    <origin xyz="0 0 0" rpy="0 0 0"/>
-    <geometry>
-      <box size="0.025 0.065 0.025"/>
-    </geometry>
-    <material name="silver_cam">
-      <color rgba="0.75 0.75 0.75 1.0"/>
-    </material>
-  </visual>
-<visual>
-    <origin xyz="0 -0.0325 0" rpy="0 0 0"/>
-    <geometry>
-      <cylinder length="0.025" radius="0.0125"/>
-    </geometry>
-    <material name="silver_cam"/>
-  </visual>
-<visual>
-    <origin xyz="0 0.0325 0" rpy="0 0 0"/>
-    <geometry>
-      <cylinder length="0.025" radius="0.0125"/>
-    </geometry>
-    <material name="silver_cam"/>
-  </visual>
-  <collision>
-    <origin xyz="0 0 0" rpy="0 0 0"/>
-    <geometry>
-      <box size="0.025 0.090 0.025"/>
-    </geometry>
-  </collision>
-  <inertial>
-    <mass value="0.072"/>
-    <inertia ixx="0.00005" ixy="0.0" ixz="0.0"
-              iyy="0.00001" iyz="0.0"
-              izz="0.00005"/>
-  </inertial>
-</link>
-<joint name="camera_joint" type="fixed">
-  <parent link="base_link"/>
-  <child link="camera_link"/>
+<xacro:depth_camera parent="base_link"
+                    update_rate="30"
+                    horizontal_fov="1.518"
+                    image_width="848"
+                    image_height="480"
+                    clip_near="0.1"
+                    clip_far="10.0"
+                    frame_id="camera_link"
+                    topic_name="camera"
+                    imu_update_rate="100"
+                    imu_topic_name="imu/data">
   <origin xyz="0.25 0.0 0.08" rpy="0 0 0"/>
-</joint>
-<link name="camera_depth_frame"></link>
-<joint name="camera_depth_joint" type="fixed">
-  <parent link="camera_link"/>
-  <child link="camera_depth_frame"/>
-  <origin xyz="0 0 0" rpy="-1.570796 0 -1.570796"/>
-</joint>
+</xacro:depth_camera>
 </robot>

Commit message: fix: simulation with slam directly

File: ros2/src/uet_amr_description/urdf/uet_amr.xacro (robot description, xacro)
@@ -3,8 +3,9 @@
     <xacro:arg name="use_real_hardware" default="false"/>
     <xacro:property name="mesh_file_scale" value="0.001 0.001 0.001"/>
-    <xacro:property name="wheel_radius" value="0.075"/>
+    <xacro:property name="wheel_radius" value="0.08255"/>
     <xacro:property name="wheel_pos_z" value="0.077157"/>
     <xacro:include filename="$(find uet_amr_description)/urdf/materials.xacro"/>
     <xacro:include filename="$(find uet_amr_description)/urdf/parts/base.xacro"/>
+    <xacro:include filename="$(find uet_amr_description)/urdf/parts/wheel.xacro"/>
     <xacro:include filename="$(find uet_amr_description)/urdf/sensors/lidar.xacro"/>
     <xacro:include filename="$(find uet_amr_description)/urdf/sensors/depth_camera.xacro"/>
@@ -27,6 +28,6 @@
         mesh_file="package://uet_amr_description/meshes/base_link.stl"
         mesh_scale="${mesh_file_scale}"
-        wheel_radius="0.075"
-        wheel_pos_z="0.077157"
+        wheel_radius="${wheel_radius}"
+        wheel_pos_z="${wheel_pos_z}"
     />
     <xacro:wheel

Commit message: chore: setup nav2, fix controller

File: ros2/src/uet_amr_description/urdf/uet_amr.xacro (robot description, xacro)
@@ -8,4 +8,5 @@
     <xacro:include filename="$(find uet_amr_description)/urdf/parts/base.xacro"/>
     <xacro:include filename="$(find uet_amr_description)/urdf/parts/wheel.xacro"/>
+    <xacro:include filename="$(find uet_amr_description)/urdf/parts/caster_wheel.xacro"/>
     <xacro:include filename="$(find uet_amr_description)/urdf/sensors/lidar.xacro"/>
     <xacro:include filename="$(find uet_amr_description)/urdf/sensors/depth_camera.xacro"/>
@@ -63,212 +64,72 @@
         joint_origin_xyz="0.002833 -0.152327 -0.078549"
     />
-    <link name="bl_caster_1">
-        <inertial>
-            <origin xyz="-0.016325683724505796 -6.209736988929682e-05 -0.02292504256915545" rpy="0 0 0"/>
-            <mass value="0.1384081385472382"/>
-            <inertia ixx="0.000106" iyy="0.00011" izz="6.3e-05" ixy="-0.0" iyz="-0.0" ixz="-3.3e-05"/>
-        </inertial>
-        <visual>
-            <origin xyz="0.213493 -0.141254 0.064203" rpy="0 0 0"/>
-            <geometry>
-                <mesh filename="package://uet_amr_description/meshes/bl_caster_1.stl" scale="0.001 0.001 0.001"/>
-            </geometry>
-            <material name="silver"/>
-        </visual>
-        <collision>
-            <origin xyz="0.213493 -0.141254 0.064203" rpy="0 0 0"/>
-            <geometry>
-                <mesh filename="package://uet_amr_description/meshes/bl_caster_1.stl" scale="0.001 0.001 0.001"/>
-            </geometry>
-        </collision>
-    </link>
-    <link name="br_caster_1">
-        <inertial>
-            <origin xyz="-0.016325165192457858 -6.199154591685074e-05 -0.02292460400344691" rpy="0 0 0"/>
-            <mass value="0.13840813854723946"/>
-            <inertia ixx="0.000106" iyy="0.00011" izz="6.3e-05" ixy="-0.0" iyz="-0.0" ixz="-3.3e-05"/>
-        </inertial>
-        <visual>
-            <origin xyz="0.212694 0.143242 0.065506" rpy="0 0 0"/>
-            <geometry>
-                <mesh filename="package://uet_amr_description/meshes/br_caster_1.stl" scale="0.001 0.001 0.001"/>
-            </geometry>
-            <material name="silver"/>
-        </visual>
-        <collision>
-            <origin xyz="0.212694 0.143242 0.065506" rpy="0 0 0"/>
-            <geometry>
-                <mesh filename="package://uet_amr_description/meshes/br_caster_1.stl" scale="0.001 0.001 0.001"/>
-            </geometry>
-        </collision>
-    </link>
-    <link name="fl_caster_1">
-        <inertial>
-            <origin xyz="-0.01632538566149161 -6.187397013268647e-05 -0.022924882170905936" rpy="0 0 0"/>
-            <mass value="0.13840813854723621"/>
-            <inertia ixx="0.000106" iyy="0.00011" izz="6.3e-05" ixy="-0.0" iyz="-0.0" ixz="-3.3e-05"/>
-        </inertial>
-        <visual>
-            <origin xyz="-0.217505 -0.142465 0.064201" rpy="0 0 0"/>
-            <geometry>
-                <mesh filename="package://uet_amr_description/meshes/fl_caster_1.stl" scale="0.001 0.001 0.001"/>
-            </geometry>
-            <material name="silver"/>
-        </visual>
-        <collision>
-            <origin xyz="-0.217505 -0.142465 0.064201" rpy="0 0 0"/>
-            <geometry>
-                <mesh filename="package://uet_amr_description/meshes/fl_caster_1.stl" scale="0.001 0.001 0.001"/>
-            </geometry>
-        </collision>
-    </link>
-    <link name="fr_caster_1">
-        <inertial>
-            <origin xyz="-0.016325867129421662 -6.17681461664299e-05 -0.022924443605240485" rpy="0 0 0"/>
-            <mass value="0.13840813854723868"/>
-            <inertia ixx="0.000106" iyy="0.00011" izz="6.3e-05" ixy="-0.0" iyz="-0.0" ixz="-3.3e-05"/>
-        </inertial>
-        <visual>
-            <origin xyz="-0.218305 0.142031 0.065504" rpy="0 0 0"/>
-            <geometry>
-                <mesh filename="package://uet_amr_description/meshes/fr_caster_1.stl" scale="0.001 0.001 0.001"/>
-            </geometry>
-            <material name="silver"/>
-        </visual>
-        <collision>
-            <origin xyz="-0.218305 0.142031 0.065504" rpy="0 0 0"/>
-            <geometry>
-                <mesh filename="package://uet_amr_description/meshes/fr_caster_1.stl" scale="0.001 0.001 0.001"/>
-            </geometry>
-        </collision>
-    </link>
-    <link name="fl_caster_wheel__1__1">
-        <inertial>
-            <origin xyz="2.5615176473869905e-05 -0.014999755176358459 -6.848949303683849e-05" rpy="0 0 0"/>
-            <mass value="0.9168727321007171"/>
-            <inertia ixx="0.000422" iyy="0.000731" izz="0.000422" ixy="-1e-06" iyz="1e-06" ixz="-0.0"/>
-        </inertial>
-        <visual>
-            <origin xyz="-0.186479 -0.157654 0.117065" rpy="0 0 0"/>
-            <geometry>
-                <mesh filename="package://uet_amr_description/meshes/fl_caster_wheel__1__1.stl" scale="0.001 0.001 0.001"/>
-            </geometry>
-            <material name="silver"/>
-        </visual>
-        <collision>
-            <origin xyz="-0.186479 -0.157654 0.117065" rpy="0 0 0"/>
-            <geometry>
-                <mesh filename="package://uet_amr_description/meshes/fl_caster_wheel__1__1.stl" scale="0.001 0.001 0.001"/>
-            </geometry>
-        </collision>
-    </link>
-    <link name="bl_caster_wheel_1">
-        <inertial>
-            <origin xyz="2.531711346762111e-05 -0.01499997857611493 -6.864989128550769e-05" rpy="0 0 0"/>
-            <mass value="0.9168727321007182"/>
-            <inertia ixx="0.000422" iyy="0.000731" izz="0.000422" ixy="-1e-06" iyz="1e-06" ixz="-0.0"/>
-        </inertial>
-        <visual>
-            <origin xyz="0.244519 -0.156443 0.117067" rpy="0 0 0"/>
-            <geometry>
-                <mesh filename="package://uet_amr_description/meshes/bl_caster_wheel_1.stl" scale="0.001 0.001 0.001"/>
-            </geometry>
-            <material name="silver"/>
-        </visual>
-        <collision>
-            <origin xyz="0.244519 -0.156443 0.117067" rpy="0 0 0"/>
-            <geometry>
-                <mesh filename="package://uet_amr_description/meshes/bl_caster_wheel_1.stl" scale="0.001 0.001 0.001"/>
-            </geometry>
-        </collision>
-    </link>
-    <link name="br_caster_wheel_1">
-        <inertial>
-            <origin xyz="-2.6164354486490904e-05 0.015000127247860873 6.878867442251801e-05" rpy="0 0 0"/>
-            <mass value="0.9168727321007177"/>
-            <inertia ixx="0.000422" iyy="0.000731" izz="0.000422" ixy="-1e-06" iyz="1e-06" ixz="-0.0"/>
-        </inertial>
-        <visual>
-            <origin xyz="0.243668 0.158053 0.118507" rpy="0 0 0"/>
-            <geometry>
-                <mesh filename="package://uet_amr_description/meshes/br_caster_wheel_1.stl" scale="0.001 0.001 0.001"/>
-            </geometry>
-            <material name="silver"/>
-        </visual>
-        <collision>
-            <origin xyz="0.243668 0.158053 0.118507" rpy="0 0 0"/>
-            <geometry>
-                <mesh filename="package://uet_amr_description/meshes/br_caster_wheel_1.stl" scale="0.001 0.001 0.001"/>
-            </geometry>
-        </collision>
-    </link>
-    <link name="fr_caster_wheel_1">
-        <inertial>
-            <origin xyz="-2.586629145395758e-05 0.014999350647611681 6.894907262748606e-05" rpy="0 0 0"/>
-            <mass value="0.9168727321007173"/>
-            <inertia ixx="0.000422" iyy="0.000731" izz="0.000422" ixy="-1e-06" iyz="1e-06" ixz="-0.0"/>
-        </inertial>
-        <visual>
-            <origin xyz="-0.18733 0.156841 0.118505" rpy="0 0 0"/>
-            <geometry>
-                <mesh filename="package://uet_amr_description/meshes/fr_caster_wheel_1.stl" scale="0.001 0.001 0.001"/>
-            </geometry>
-            <material name="silver"/>
-        </visual>
-        <collision>
-            <origin xyz="-0.18733 0.156841 0.118505" rpy="0 0 0"/>
-            <geometry>
-                <mesh filename="package://uet_amr_description/meshes/fr_caster_wheel_1.stl" scale="0.001 0.001 0.001"/>
-            </geometry>
-        </collision>
-    </link>
-    <joint name="Revolute 19" type="continuous">
-        <origin xyz="-0.213493 0.141254 -0.064203" rpy="0 0 0"/>
-        <parent link="base_link"/>
-        <child link="bl_caster_1"/>
-        <axis xyz="-8e-06 0.004578 -0.99999"/>
-    </joint>
-    <joint name="Revolute 20" type="continuous">
-        <origin xyz="-0.212694 -0.143242 -0.065506" rpy="0 0 0"/>
-        <parent link="base_link"/>
-        <child link="br_caster_1"/>
-        <axis xyz="-8e-06 0.004578 -0.99999"/>
-    </joint>
-    <joint name="Revolute 21" type="continuous">
-        <origin xyz="0.217505 0.142465 -0.064201" rpy="0 0 0"/>
-        <parent link="base_link"/>
-        <child link="fl_caster_1"/>
-        <axis xyz="-8e-06 0.004578 -0.99999"/>
-    </joint>
-    <joint name="Revolute 22" type="continuous">
-        <origin xyz="0.218305 -0.142031 -0.065504" rpy="0 0 0"/>
-        <parent link="base_link"/>
-        <child link="fr_caster_1"/>
-        <axis xyz="-8e-06 0.004578 -0.99999"/>
-    </joint>
-    <joint name="Revolute 23" type="continuous">
-        <origin xyz="-0.031026 0.015189 -0.052864" rpy="0 0 0"/>
-        <parent link="fl_caster_1"/>
-        <child link="fl_caster_wheel__1__1"/>
-        <axis xyz="0.001715 -0.999988 -0.004578"/>
-    </joint>
-    <joint name="Revolute 24" type="continuous">
-        <origin xyz="-0.031026 0.015189 -0.052864" rpy="0 0 0"/>
-        <parent link="bl_caster_1"/>
-        <child link="bl_caster_wheel_1"/>
-        <axis xyz="0.001715 -0.999988 -0.004578"/>
-    </joint>
-    <joint name="Revolute 25" type="continuous">
-        <origin xyz="-0.030974 -0.014811 -0.053001" rpy="0 0 0"/>
-        <parent link="br_caster_1"/>
-        <child link="br_caster_wheel_1"/>
-        <axis xyz="0.001715 -0.999988 -0.004578"/>
-    </joint>
-    <joint name="Revolute 26" type="continuous">
-        <origin xyz="-0.030975 -0.01481 -0.053001" rpy="0 0 0"/>
-        <parent link="fr_caster_1"/>
-        <child link="fr_caster_wheel_1"/>
-        <axis xyz="0.001715 -0.999988 -0.004578"/>
-    </joint>
+    <xacro:caster
+        corner="bl" parent="base_link" mesh_scale="${mesh_file_scale}"
+        mount_mass="0.1384081385472382"
+        mount_inertial_origin_xyz="-0.016325683724505796 -6.209736988929682e-05 -0.02292504256915545"
+        mount_ixx="0.000106" mount_iyy="0.00011" mount_izz="6.3e-05" mount_ixy="-0.0" mount_iyz="-0.0" mount_ixz="-3.3e-05"
+        mount_visual_origin_xyz="0.213493 -0.141254 0.064203"
+        mount_mesh_file="package://uet_amr_description/meshes/bl_caster_1.stl"
+        mount_joint_origin_xyz="-0.213493 0.141254 -0.064203"
+        mount_joint_axis="-8e-06 0.004578 -0.99999"
+        wheel_mass="0.9168727321007182"
+        wheel_inertial_origin_xyz="2.531711346762111e-05 -0.01499997857611493 -6.864989128550769e-05"
+        wheel_ixx="0.000422" wheel_iyy="0.000731" wheel_izz="0.000422" wheel_ixy="-1e-06" wheel_iyz="1e-06" wheel_ixz="-0.0"
+        wheel_visual_origin_xyz="0.244519 -0.156443 0.117067"
+        wheel_mesh_file="package://uet_amr_description/meshes/bl_caster_wheel_1.stl"
+        wheel_joint_origin_xyz="-0.031026 0.015189 -0.052864"
+        wheel_joint_axis="0.001715 -0.999988 -0.004578"
+    />
+    <xacro:caster
+        corner="br" parent="base_link" mesh_scale="${mesh_file_scale}"
+        mount_mass="0.13840813854723946"
+        mount_inertial_origin_xyz="-0.016325165192457858 -6.199154591685074e-05 -0.02292460400344691"
+        mount_ixx="0.000106" mount_iyy="0.00011" mount_izz="6.3e-05" mount_ixy="-0.0" mount_iyz="-0.0" mount_ixz="-3.3e-05"
+        mount_visual_origin_xyz="0.212694 0.143242 0.065506"
+        mount_mesh_file="package://uet_amr_description/meshes/br_caster_1.stl"
+        mount_joint_origin_xyz="-0.212694 -0.143242 -0.065506"
+        mount_joint_axis="-8e-06 0.004578 -0.99999"
+        wheel_mass="0.9168727321007177"
+        wheel_inertial_origin_xyz="-2.6164354486490904e-05 0.015000127247860873 6.878867442251801e-05"
+        wheel_ixx="0.000422" wheel_iyy="0.000731" wheel_izz="0.000422" wheel_ixy="-1e-06" wheel_iyz="1e-06" wheel_ixz="-0.0"
+        wheel_visual_origin_xyz="0.243668 0.158053 0.118507"
+        wheel_mesh_file="package://uet_amr_description/meshes/br_caster_wheel_1.stl"
+        wheel_joint_origin_xyz="-0.030974 -0.014811 -0.053001"
+        wheel_joint_axis="0.001715 -0.999988 -0.004578"
+    />
+    <xacro:caster
+        corner="fl" parent="base_link" mesh_scale="${mesh_file_scale}"
+        mount_mass="0.13840813854723621"
+        mount_inertial_origin_xyz="-0.01632538566149161 -6.187397013268647e-05 -0.022924882170905936"
+        mount_ixx="0.000106" mount_iyy="0.00011" mount_izz="6.3e-05" mount_ixy="-0.0" mount_iyz="-0.0" mount_ixz="-3.3e-05"
+        mount_visual_origin_xyz="-0.217505 -0.142465 0.064201"
+        mount_mesh_file="package://uet_amr_description/meshes/fl_caster_1.stl"
+        mount_joint_origin_xyz="0.217505 0.142465 -0.064201"
+        mount_joint_axis="-8e-06 0.004578 -0.99999"
+        wheel_mass="0.9168727321007171"
+        wheel_inertial_origin_xyz="2.5615176473869905e-05 -0.014999755176358459 -6.848949303683849e-05"
+        wheel_ixx="0.000422" wheel_iyy="0.000731" wheel_izz="0.000422" wheel_ixy="-1e-06" wheel_iyz="1e-06" wheel_ixz="-0.0"
+        wheel_visual_origin_xyz="-0.186479 -0.157654 0.117065"
+        wheel_mesh_file="package://uet_amr_description/meshes/fl_caster_wheel__1__1.stl"
+        wheel_joint_origin_xyz="-0.031026 0.015189 -0.052864"
+        wheel_joint_axis="0.001715 -0.999988 -0.004578"
+    />
+    <xacro:caster
+        corner="fr" parent="base_link" mesh_scale="${mesh_file_scale}"
+        mount_mass="0.13840813854723868"
+        mount_inertial_origin_xyz="-0.016325867129421662 -6.17681461664299e-05 -0.022924443605240485"
+        mount_ixx="0.000106" mount_iyy="0.00011" mount_izz="6.3e-05" mount_ixy="-0.0" mount_iyz="-0.0" mount_ixz="-3.3e-05"
+        mount_visual_origin_xyz="-0.218305 0.142031 0.065504"
+        mount_mesh_file="package://uet_amr_description/meshes/fr_caster_1.stl"
+        mount_joint_origin_xyz="0.218305 -0.142031 -0.065504"
+        mount_joint_axis="-8e-06 0.004578 -0.99999"
+        wheel_mass="0.9168727321007173"
+        wheel_inertial_origin_xyz="-2.586629145395758e-05 0.014999350647611681 6.894907262748606e-05"
+        wheel_ixx="0.000422" wheel_iyy="0.000731" wheel_izz="0.000422" wheel_ixy="-1e-06" wheel_iyz="1e-06" wheel_ixz="-0.0"
+        wheel_visual_origin_xyz="-0.18733 0.156841 0.118505"
+        wheel_mesh_file="package://uet_amr_description/meshes/fr_caster_wheel_1.stl"
+        wheel_joint_origin_xyz="-0.030975 -0.01481 -0.053001"
+        wheel_joint_axis="0.001715 -0.999988 -0.004578"
+    />
     <xacro:lidar
         frame_id="front_lidar"

Commit message: fix: rotate yaw of lidar in real robot 180 degrees

File: ros2/src/uet_amr_description/urdf/uet_amr.xacro (robot description, xacro)
@@ -17,4 +17,8 @@
         <xacro:include filename="$(find uet_amr_description)/urdf/uet_amr.ros2control"/>
     </xacro:unless>
+    <xacro:property name="front_lidar_yaw" value="0"/>
+    <xacro:if value="$(arg use_real_hardware)">
+        <xacro:property name="front_lidar_yaw" value="3.14159"/>
+    </xacro:if>
     <xacro:include filename="$(find uet_amr_description)/urdf/uet_amr.gazebo"/>
     <xacro:base
@@ -143,5 +147,5 @@
         max_range="25.0"
     >
-        <origin xyz="0.25 -0.16 0.088" rpy="0 0 0"/>
+        <origin xyz="0.25 -0.16 0.088" rpy="0 0 ${front_lidar_yaw}"/>
     </xacro:lidar>
     <!-- Rear lidar will be added later.

Commit message: fix: orin nx real test

File: ros2/src/uet_amr_description/urdf/uet_amr.xacro (robot description, xacro)
@@ -176,5 +176,10 @@
         imu_update_rate="200"
         imu_topic_name="camera/camera/imu">
-        <origin xyz="0.25 0.0 0.08" rpy="0 0 0"/>
+        <!-- Calibrated against the floor: depth points transformed through this TF must land on
+             z = 0 at every range. Lens 0.215 m above the floor (base_link is 0.005 m above
+             base_footprint, which is on the floor), tilted 1.9 deg DOWN (positive URDF pitch).
+             Any pitch error shows up as floor rising with distance, ~10 cm at 3 m for 2 deg, which
+             nvblox turns into phantom obstacles. -->
+        <origin xyz="0.25 0.0 0.210" rpy="0 0.033 0"/>
     </xacro:depth_camera>
 </robot>
